File: hardware/kicad/power.kicad_sch (KiCad schematic)
At the start: 18 parts, among them Q1 AO3401A (reverse battery), Q2 AO3401A (load share), U2 MCP73831T-2ACI/OT, U3 AP2112K-3.3TRG1

Commit message: Roadmap: $2,000 budget plan and $225 + $15/month pricing
Adds a money section to the launch roadmap: how the starting budget is
split into two supply waves, profit per unit and per subscriber, and how
preorders compound into bigger batches. Also saves the PR description.

Co-Authored-By: Claude Opus 5.5 <noreply@anthropic.com>
Parts:
- U3: value AP2112K-3.3TRG1 -> RT9080-33GJ5; LCSC C51118 -> C841192
Connections:
- net +3V3: no longer R20.1
- net VBUS_SENSE: now also R20.1
Changed lines of the file:
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@@
 			)
 		)
-		(property "Value" "AP2112K-3.3TRG1"
+		(property "Value" "RT9080-33GJ5"
 			(at 190.5 69.85 0)
 			(show_name no)
@@
 			)
 		)
-		(property "Datasheet" "https://www.diodes.com/assets/Datasheets/AP2112.pdf"
+		(property "Datasheet" "https://www.richtek.com/assets/product_file/RT9080/DS9080-09.pdf"
 			(at 190.5 62.23 0)
 			(hide yes)
@@
 			)
 		)
-		(property "Description" "600mA low dropout linear regulator, with enable pin, 3.8V-6V input voltage range, 3.3V fixed positive output, SOT-23-5"
+		(property "Description" "600mA low-Iq (2uA) LDO, 3.3V fixed, VIN 1.2-5.5V, TSOT-23-5 (1 VIN, 2 GND, 3 EN, 4 NC, 5 VOUT, same as AP2112K)"
 			(at 190.5 59.69 0)
 			(hide yes)
@@
 			)
 		)
-		(property "LCSC" "C51118"
+		(property "LCSC" "C841192"
 			(at 190.5 59.69 0)
 			(hide yes)
@@
 		)
 	)
-	(global_label "+3V3"
+	(global_label "VBUS_SENSE"
 		(at 110.49 135.89 90)
 		(effects
