File: hardware/kicad/keypad.kicad_sch (KiCad schematic)
At the start: 57 parts, among them SW1 SHIFT, SW10 x^2, SW11 x^n, SW12 log, SW13 ln, SW14 (-), SW15 deg-min-sec, SW16 hyp, SW17 sin, SW18 cos, SW19 tan, SW2 ALPHA, SW20 RCL, SW21 ENG, SW22 (, SW23 ), SW24 S<>D, SW25 M+, SW26 7, SW27 8, SW28 9, SW29 DEL, SW3 MODE, SW30 AC, SW31 4, SW32 5, SW33 6, SW34 x, SW35 /, SW36 1, SW37 2, SW38 3, SW39 +, SW4 Abs, SW40 -, SW41 0, SW42 ., SW43 x10^x, SW44 Ans, SW45 =, SW46 UP, SW47 DOWN, SW48 LEFT, SW49 RIGHT, SW5 x^3, SW50 ON, SW6 x^-1, SW7 log_a, SW8 a/b, SW9 sqrt, U6 TCA8418RTWR

Commit message: Final review, v14 order prep, firmware fixes and production planning
- PCB v14 confirmed GO by final reviews (verification 06, 08, 11)
- CAD fit rev G with measured rib/pin/hook heights; grind zones 6, 6b, 6c
- Firmware: OTA updates, phone setup portal, low-battery gate, polish
- Docs: arrival checklist, vendor comparison, order walkthrough updates
- Production: QA test plan, knockoff shell plan, cost model

Co-Authored-By: Claude Opus 5.5 <noreply@anthropic.com>
Parts:
- SW1: footprint ai_calc:KeyPad_6.0x4.5 -> ai_calc:KeyPad_6.0x4.5_H3notch
- SW4: value Abs -> CALC
- SW5: value x^3 -> ∫dx
Changed lines of the file:
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@@
 			)
 		)
-		(property "Footprint" "ai_calc:KeyPad_6.0x4.5"
+		(property "Footprint" "ai_calc:KeyPad_6.0x4.5_H3notch"
 			(at 39.37 100.33 0)
 			(hide yes)
@@
 			)
 		)
-		(property "Value" "Abs"
+		(property "Value" "CALC"
 			(at 184.15 111.76 0)
 			(show_name no)
@@
 			)
 		)
-		(property "Value" "x^3"
+		(property "Value" "∫dx"
 			(at 208.28 111.76 0)
 			(show_name no)
